Commit message: Glider LHS verified compared to MATLAB results using hard-coded inputs

File: glider_hybrid_whoi_description/urdf/glider_hybrid_whoi_base_test.xacro (robot description, xacro)
@@ -16,13 +16,14 @@
   <xacro:include filename="$(find uuv_descriptions)/urdf/common.urdf.xacro" />
   <xacro:include filename="$(find uuv_sensor_ros_plugins)/urdf/sensor_snippets.xacro"/>
-  <xacro:include filename="$(find glider_hybrid_whoi_description)/urdf/glider_hybrid_whoi_snippets.xacro"/>
+  <xacro:include filename="$(find glider_hybrid_whoi_description)/urdf/glider_hybrid_whoi_snippets_test.xacro"/>
   <xacro:include filename="$(find uuv_gazebo_ros_plugins)/urdf/snippets.xacro"/>
   <!-- Properties -->
-  <xacro:property name="mass" value="69.7"/>
-  <xacro:property name="hull_mass" value="60.4"/>
-  <xacro:property name="shifter_mass" value="9.3"/>
-  <xacro:property name="length" value="1.98"/>
-  <xacro:property name="diameter" value="0.23"/>
-  <xacro:property name="radius" value="${diameter*0.5}"/>
+  <xacro:property name="mass" value="56.0"/>
+  <xacro:property name="hull_mass" value="48.2"/>
+  <xacro:property name="shifter_mass" value="7.8"/>
+  <xacro:property name="length" value="2.0"/>
+  <xacro:property name="radius" value="0.105"/>
+  <xacro:property name="diameter" value="${radius*2}"/>
+  <xacro:property name="area" value="${radius*radius*3.141592}"/>
   <xacro:property name="ballast_tank_radius" value="0.07"/>
   <xacro:property name="initial_mass_pos" value="0.4"/>
@@ -30,10 +31,8 @@
   <xacro:property name="max_mass_pos" value="0.03"/>
   <xacro:property name="max_ballast_vol" value="2.4e-04"/>
-  <xacro:property name="volume" value="0.06799987704121499"/> <!--usage?-->
+  <xacro:property name="volume" value="99999999"/> <!-- usage? Neutural buoyancy disabled using zero gravity world-->
   <xacro:property name="cob" value="0 0 0"/>
   <xacro:property name="cog" value="0 0 0.0054"/>
-  <xacro:property name="rho" value="1027.0"/>
-  <xacro:property name="area" value="0.04155"/>
-  <xacro:property name="length" value="1.98"/>
+  <xacro:property name="rho" value="1024.0"/>
   <!-- <xacro:property name="visual_mesh_file" value="file://$(find glider_hybrid_whoi_description)/mesh/glider_hybrid_whoi.dae"/>
   <xacro:property name="collision_mesh_file" value="file://$(find glider_hybrid_whoi_description)/mesh/glider_hybrid_whoi_collision.dae"/>
@@ -45,4 +44,6 @@
   <xacro:property name="fin_mesh_file" value="file://$(find glider_hybrid_whoi_description)/mesh/eca_a9/eca_a9_fin.dae"/>
   <xacro:macro name="glider_hybrid_whoi_base" params="namespace debug inertial_reference_frame">
+    <!-- <link name="dummy">
+    </link> -->
     <link name="${namespace}/base_link">
       <visual>
@@ -58,12 +59,18 @@
         </geometry>
       </collision>
+      <!-- This inertial input is dummy input. The values will be changed within glider kinamatics plugin with Fossen's-->
       <inertial>
+        <origin xyz="0 0 0" rpy="0 0 0"/>
         <mass value="${mass}" />
-        <origin xyz="0 0 0" rpy="0 0 0"/>
-        <inertia ixx="0.6" ixy="0" ixz="0"
-                 iyy="30.0" iyz="0"
-                 izz="35.0" />
+        <inertia ixx="0.3048" ixy="0" ixz="0"
+                 iyy="13.9760" iyz="0"
+                 izz="13.9760" />
       </inertial>
     </link>
+    <!-- Dummy joint to fix inertial definition at urdf warnings -->
+    <!-- <joint name="dummy_joint" type="fixed">
+      <parent link="dummy"/>
+      <child link="${namespace}/base_link"/>
+    </joint> -->
     <!-- Set up hydrodynamic plugin -->
     <gazebo>
@@ -72,29 +79,37 @@
         <flow_velocity_topic>hydrodynamics/current_velocity</flow_velocity_topic>
         <debug>${debug}</debug>
-        <writeLog>0</writeLog>
+        <writeLog>1</writeLog>
         <link name="${namespace}/base_link">
           <volume>${volume}</volume>
           <center_of_buoyancy>${cob}</center_of_buoyancy>
           <center_of_gravity>${cog}</center_of_gravity>
-          <neutrally_buoyant>1</neutrally_buoyant>
-          <hard_code_input>0</hard_code_input>
+          <neutrally_buoyant>0</neutrally_buoyant>
+          <hard_code_input>1</hard_code_input>
           <hydrodynamic_model>
             <type>fossen</type>
-            <added_mass>
-              4   0   0   0   0   0
-              0   95  0   0   0   0
-              0   0   75  0   0   0
-              0   0   0   0.4 0   0
-              0   0   0   0   27  0
-              0   0   0   0   0   32
+            <added_mass> <!-- dummy input. The values will be changed within glider kinamatics plugin-->
+              100 0   0   0   0   0
+              0   100 0   0   0   0
+              0   0   100 0   0   0
+              0   0   0   100 0   0
+              0   0   0   0   100 0
+              0   0   0   0   0   100
             </added_mass>
-            <linear_damping_forward_speed>
-              -8      0       0       0       0       0
-              0       -162    0       0       0       150
-              0       0       -108    0       -100    0
-              0       0       0       -13     0       0
-              0       0       37      0       -20     0
-              0       -34     0       0       0       -32
-            </linear_damping_forward_speed>
+            <!-- <linear_damping_forward_speed>
+              0       0       0       0       0       0
+              0       0       0       0       0       0
+              0       0       -14     0       0       0
+              0       0       0       0       0       0
+              0       0       0       0       -12     0
+              0       0       0       0       0       0
+            </linear_damping_forward_speed> -->
+            <linear_damping>
+              0       0       0       0       0       0
+              0       0       0       0       0       0
+              0       0       -14     0       0       0
+              0       0       0       0       0       0
+              0       0       0       0       -12     0
+              0       0       0       0       0       0
+            </linear_damping>
           </hydrodynamic_model>
             <ballast_radius>${ballast_tank_radius}</ballast_radius>
@@ -111,10 +126,10 @@
     </gazebo>
     <!-- Instantiate Fins -->
-    <xacro:fin_macro namespace="${namespace}" fin_id="0">
+    <!-- <xacro:fin_macro namespace="${namespace}" fin_id="0">
       <origin xyz="-0.70777 -0.07876 0.078586" rpy="0.7904 -0.0998 -0.1003" />
     </xacro:fin_macro>
     <xacro:fin_macro namespace="${namespace}" fin_id="1">
       <origin xyz="-0.70777 -0.07876 -0.078586" rpy="2.3512 0.0998 -0.1003" />
-    </xacro:fin_macro>
+    </xacro:fin_macro> -->
     <!--
     <xacro:fin_macro namespace="${namespace}" fin_id="2">
@@ -125,14 +140,14 @@
     </xacro:fin_macro>
     -->
-    <xacro:thruster_module_first_order_basic_fcn_macro
+    <!-- <xacro:thruster_module_first_order_basic_fcn_macro
       namespace="${namespace}"
       thruster_id="0"
       mesh_filename="${prop_mesh_file}"
       dyn_time_constant="0.1"
-      rotor_constant="0.000049">
+      rotor_constant="0.00049">
       <origin xyz="-0.9676 0 0" rpy="0 0 ${pi}" />
-    </xacro:thruster_module_first_order_basic_fcn_macro>
+    </xacro:thruster_module_first_order_basic_fcn_macro> -->
     <!-- TODO: Parametrize the battery unit -->
-    <xacro:basic_linear_battery_macro
+    <!-- <xacro:basic_linear_battery_macro
       namespace="${namespace}"
       parent_link="${namespace}/base_link"
@@ -145,6 +160,6 @@
       smooth_current_tau="1.9499"
       voltage="4.2"
-      update_rate="2.0"/>
-    <xacro:include filename="$(find glider_hybrid_whoi_description)/urdf/glider_hybrid_whoi_sensors.xacro"/>
+      update_rate="2.0"/> -->
+    <xacro:include filename="$(find glider_hybrid_whoi_description)/urdf/glider_hybrid_whoi_sensors_test.xacro"/>
   </xacro:macro>
 </robot>
