Commit message: re-added ECA A9 for example visual vehicle (using whoi glider require more specifications for sensor locations) and added simple passing through pipeline plugins for BuoyancyPump and SlidingMass

File: glider_hybrid_whoi_description/urdf/glider_hybrid_whoi_base.xacro (robot description, xacro)
@@ -28,8 +28,12 @@
   <xacro:property name="area" value="0.04155"/>
   <xacro:property name="length" value="1.98"/>
-  <xacro:property name="visual_mesh_file" value="file://$(find glider_hybrid_whoi_description)/mesh/glider_hybrid_whoi.dae"/>
+  <!-- <xacro:property name="visual_mesh_file" value="file://$(find glider_hybrid_whoi_description)/mesh/glider_hybrid_whoi.dae"/>
   <xacro:property name="collision_mesh_file" value="file://$(find glider_hybrid_whoi_description)/mesh/glider_hybrid_whoi_collision.dae"/>
   <xacro:property name="prop_mesh_file" value="file://$(find glider_hybrid_whoi_description)/mesh/glider_hybrid_whoi_propeller.dae"/>
-  <xacro:property name="fin_mesh_file" value="file://$(find glider_hybrid_whoi_description)/mesh/glider_hybrid_whoi_fin.dae"/>
+  <xacro:property name="fin_mesh_file" value="file://$(find glider_hybrid_whoi_description)/mesh/glider_hybrid_whoi_fin.dae"/> -->
+  <xacro:property name="visual_mesh_file" value="file://$(find glider_hybrid_whoi_description)/mesh/eca_a9/eca_a9.dae"/>
+  <xacro:property name="collision_mesh_file" value="file://$(find glider_hybrid_whoi_description)/mesh/eca_a9/eca_a9.stl"/>
+  <xacro:property name="prop_mesh_file" value="file://$(find glider_hybrid_whoi_description)/mesh/eca_a9/eca_a9_propeller.dae"/>
+  <xacro:property name="fin_mesh_file" value="file://$(find glider_hybrid_whoi_description)/mesh/eca_a9/eca_a9_fin.dae"/>
   <xacro:macro name="glider_hybrid_whoi_base" params="namespace debug inertial_reference_frame">
     <link name="${namespace}/base_link">

Commit message: fixed jumping out of water problem. Still, it is slowly drawning

File: glider_hybrid_whoi_description/urdf/glider_hybrid_whoi_base.xacro (robot description, xacro)
@@ -20,4 +20,6 @@
   <!-- Properties -->
   <xacro:property name="mass" value="69.7"/>
+  <xacro:property name="hull_mass" value="60.4"/>
+  <xacro:property name="shifter_mass" value="9.3"/>
   <xacro:property name="length" value="1.98"/>
   <xacro:property name="diameter" value="0.23"/>
@@ -67,5 +69,5 @@
           <volume>${volume}</volume>
           <center_of_buoyancy>${cob}</center_of_buoyancy>
-          <neutrally_buoyant>0</neutrally_buoyant>
+          <neutrally_buoyant>1</neutrally_buoyant>
           <hydrodynamic_model>
             <type>fossen</type>
@@ -90,6 +92,6 @@
             <hull_length>${length}</hull_length>
             <hull_radius>${radius}</hull_radius>
-            <hull_mass>${mass}</hull_mass>
-            <shifter_mass>9.3</shifter_mass>
+            <hull_mass>${hull_mass}</hull_mass>
+            <shifter_mass>${shifter_mass}</shifter_mass>
             <initial_mass_position>0.04</initial_mass_position>
             <initial_ballast_position>0.06</initial_ballast_position>

Commit message: add gitignore for vscode profiles and clean basic launch set-ups for kinematics testings

File: glider_hybrid_whoi_description/urdf/glider_hybrid_whoi_base.xacro (robot description, xacro)
@@ -67,5 +67,5 @@
     </link>
     <!-- Set up hydrodynamic plugin -->
-    <gazebo>
+    <!-- <gazebo>
       <plugin name="${namespace}_hybrid_glider_plugin" filename="libhybrid_glider_underwater_object_ros_plugin.so">
         <fluid_density>${rho}</fluid_density>
@@ -109,12 +109,12 @@
         </link>
       </plugin>
-    </gazebo>
+    </gazebo> -->
     <!-- Instantiate Fins -->
-    <xacro:fin_macro namespace="${namespace}" fin_id="0">
+    <!-- <xacro:fin_macro namespace="${namespace}" fin_id="0">
       <origin xyz="-0.70777 -0.07876 0.078586" rpy="0.7904 -0.0998 -0.1003" />
     </xacro:fin_macro>
     <xacro:fin_macro namespace="${namespace}" fin_id="1">
       <origin xyz="-0.70777 -0.07876 -0.078586" rpy="2.3512 0.0998 -0.1003" />
-    </xacro:fin_macro>
+    </xacro:fin_macro> -->
     <!--
     <xacro:fin_macro namespace="${namespace}" fin_id="2">
@@ -125,5 +125,5 @@
     </xacro:fin_macro>
     -->
-    <xacro:thruster_module_first_order_basic_fcn_macro
+    <!-- <xacro:thruster_module_first_order_basic_fcn_macro
       namespace="${namespace}"
       thruster_id="0"
@@ -132,7 +132,7 @@
       rotor_constant="0.000049">
       <origin xyz="-0.9676 0 0" rpy="0 0 ${pi}" />
-    </xacro:thruster_module_first_order_basic_fcn_macro>
+    </xacro:thruster_module_first_order_basic_fcn_macro> -->
     <!-- TODO: Parametrize the battery unit -->
-    <xacro:basic_linear_battery_macro
+    <!-- <xacro:basic_linear_battery_macro
       namespace="${namespace}"
       parent_link="${namespace}/base_link"
@@ -145,5 +145,5 @@
       smooth_current_tau="1.9499"
       voltage="4.2"
-      update_rate="2.0"/>
+      update_rate="2.0"/> -->
     <xacro:include filename="$(find glider_hybrid_whoi_description)/urdf/glider_hybrid_whoi_sensors.xacro"/>
   </xacro:macro>

File: glider_hybrid_whoi_description/urdf/glider_hybrid_whoi_sensors.xacro (robot description, xacro)
@@ -31,20 +31,20 @@
       <origin xyz="0.4785 0.0 -0.0825" rpy="0 ${0.5*pi} 0" />
     </xacro:dvl_plugin_macro>
-    <xacro:switchable_battery_consumer_macro
+    <!-- <xacro:switchable_battery_consumer_macro
       link_name="${namespace}/dvl_link"
       battery_link="${namespace}/battery_link"
       battery_name="${namespace}/battery"
       power_load="25"
-      topic="${namespace}/dvl/state"/>
+      topic="${namespace}/dvl/state"/> -->
     <!-- Side scan sonar left -->
     <xacro:sidescan_sonar namespace="${namespace}" parent_link="${namespace}/base_link" suffix="left">
       <origin xyz="0.41225 0.1498 -0.04615" rpy="${0.5*pi} ${-5*d2r+pi/3.0} ${0.5*pi}" />
     </xacro:sidescan_sonar>
-    <xacro:switchable_battery_consumer_macro
+    <!-- <xacro:switchable_battery_consumer_macro
       link_name="${namespace}/sonarleft_link"
       battery_link="${namespace}/battery_link"
       battery_name="${namespace}/battery"
       power_load="25"
-      topic="${namespace}/sonarleft/state"/>
+      topic="${namespace}/sonarleft/state"/> -->
     <!-- Side scan sonar right -->
     <xacro:sidescan_sonar
@@ -52,10 +52,10 @@
       <origin xyz="0.41225 -0.1498 -0.04615" rpy="${0.5*pi} ${-5*d2r+pi/3.0} ${-0.5*pi}" />
     </xacro:sidescan_sonar>
-    <xacro:switchable_battery_consumer_macro
+    <!-- <xacro:switchable_battery_consumer_macro
       link_name="${namespace}/sonarright_link"
       battery_link="${namespace}/battery_link"
       battery_name="${namespace}/battery"
       power_load="25"
-      topic="${namespace}/sonarright/state"/>
+      topic="${namespace}/sonarright/state"/> -->
     <!-- RPT
     <xacro:default_rpt namespace="${namespace}" parent_link="${namespace}/base_link">
@@ -66,20 +66,20 @@
       <origin xyz="0 0 0" rpy="0 0 0"/>
     </xacro:default_pressure>
-    <xacro:switchable_battery_consumer_macro
+    <!-- <xacro:switchable_battery_consumer_macro
       link_name="${namespace}/pressure_link"
       battery_link="${namespace}/battery_link"
       battery_name="${namespace}/battery"
       power_load="5"
-      topic="${namespace}/pressure/state"/>
+      topic="${namespace}/pressure/state"/> -->
     <!-- IMU  -->
     <xacro:default_imu namespace="${namespace}" parent_link="${namespace}/base_link">
       <origin xyz="0 0 0" rpy="0 0 0"/>
     </xacro:default_imu>
-    <xacro:switchable_battery_consumer_macro
+    <!-- <xacro:switchable_battery_consumer_macro
       link_name="${namespace}/imu_link"
       battery_link="${namespace}/battery_link"
       battery_name="${namespace}/battery"
       power_load="20"
-      topic="${namespace}/imu/state"/>
+      topic="${namespace}/imu/state"/> -->
     <!-- Mount a camera -->
     <xacro:regular_camera_plugin_macro
@@ -98,21 +98,21 @@
         <origin xyz="-0.375 0 -0.16" rpy="0 0.3 0"/>
     </xacro:regular_camera_plugin_macro>
-    <xacro:switchable_battery_consumer_macro
+    <!-- <xacro:switchable_battery_consumer_macro
       link_name="${namespace}/camera_link"
       battery_link="${namespace}/battery_link"
       battery_name="${namespace}/battery"
       power_load="25"
-      topic=""/>
+      topic=""/> -->
     <!-- Mount a GPS. -->
     <xacro:default_gps namespace="${namespace}" parent_link="${namespace}/base_link" />
-    <xacro:switchable_battery_consumer_macro
+    <!-- <xacro:switchable_battery_consumer_macro
       link_name="${namespace}/gps_link"
       battery_link="${namespace}/battery_link"
       battery_name="${namespace}/battery"
       power_load="5"
-      topic=""/>
+      topic=""/> -->
     <!-- Mount the chemical concentration sensor -->
-    <xacro:default_chemical_concentration_sensor namespace="${namespace}" parent_link="${namespace}/base_link">
+    <!-- <xacro:default_chemical_concentration_sensor namespace="${namespace}" parent_link="${namespace}/base_link">
       <origin xyz="0 0 0" rpy="0 0 0"/>
-    </xacro:default_chemical_concentration_sensor>
+    </xacro:default_chemical_concentration_sensor> -->
 </robot>

File: glider_hybrid_whoi_description/urdf/glider_hybrid_whoi_snippets.xacro (robot description, xacro)
@@ -18,5 +18,5 @@
     <xacro:property name="fin_rho" value="1028.0"/>
     <!-- FIN SNIPPETS -->
-    <xacro:macro name="fin_macro" params="namespace fin_id *origin">
+    <!-- <xacro:macro name="fin_macro" params="namespace fin_id *origin">
       <xacro:fin_two_lines_macro
         namespace="${namespace}"
@@ -38,5 +38,5 @@
         <xacro:insert_block name="origin"/>
       </xacro:fin_two_lines_macro>
-    </xacro:macro>
+    </xacro:macro> -->
     <!-- <xacro:macro name="fin_macro" params="namespace fin_id *origin">
       <xacro:fin_quadratic_macro
