Commit message: fixes after rebase

File: glider_hybrid_whoi_description/urdf/glider_asv_base_kinematics.xacro (robot description, xacro)
@@ -29,5 +29,5 @@
     <link name="${namespace}/base_link">
       <visual>
-        <origin xyz="0 0 0" rpy="0 0 0" />
+        <origin xyz="0 0 0" rpy="0 0 ${pi/2}" />
         <geometry>
           <mesh filename="${visual_mesh_file}" scale="1 1 1" />
@@ -35,5 +35,5 @@
       </visual>
       <collision>
-        <origin xyz="0 0 0" rpy="0 0 0" />
+        <origin xyz="0 0 0" rpy="0 0 ${pi/2}" />
         <geometry>
           <mesh filename="${collision_mesh_file}" scale="1 1 1" />
@@ -42,5 +42,5 @@
       <inertial>
         <mass value="${mass}"/>
-        <origin xyz="0 0 0" rpy="0 0 0" />
+        <origin xyz="0 0 0" rpy="0 0 ${pi/2}" />
         <inertia ixx="0.3048" ixy="0" ixz="0" iyy="13.976" iyz="0" izz="13.976" />
       </inertial>
@@ -56,4 +56,5 @@
         <espg_projection>26987</espg_projection>
         <!-- Kinematics coefficients -->
+        <surface_vehicle>true</surface_vehicle>
         <f_pitch_battpos_cal_m>1.2565</f_pitch_battpos_cal_m>
         <f_pitch_battpos_cal_b>-0.055</f_pitch_battpos_cal_b>

Commit message: rewrite ASV code and examples

File: glider_hybrid_whoi_description/urdf/glider_asv_base_kinematics.xacro (robot description, xacro)
@@ -23,13 +23,11 @@
   <xacro:property name="cob" value="0 0 0"/>
   <xacro:property name="cog" value="0 0 0.0054"/>
-  <xacro:property name="visual_mesh_file" value="file://$(find glider_hybrid_whoi_description)/mesh/glider_hybrid_whoi/glider_hybrid_whoi_body.dae" />
-  <xacro:property name="collision_mesh_file" value="file://$(find glider_hybrid_whoi_description)/mesh/glider_hybrid_whoi/glider_hybrid_whoi_collision.dae" />
-  <xacro:property name="left_prop_mesh_file" value="file://$(find glider_hybrid_whoi_description)/mesh/glider_hybrid_whoi/glider_hybrid_whoi_left_propeller.dae" />
-  <xacro:property name="right_prop_mesh_file" value="file://$(find glider_hybrid_whoi_description)/mesh/glider_hybrid_whoi/glider_hybrid_whoi_right_propeller.dae" />
-  <xacro:macro name="glider_hybrid_whoi_base" params="namespace debug inertial_reference_frame">
+  <xacro:property name="visual_mesh_file" value="file://$(find glider_hybrid_whoi_description)/mesh/glider_asv/Wave Glider-Float.dae" />
+  <xacro:property name="collision_mesh_file" value="file://$(find glider_hybrid_whoi_description)/mesh/glider_asv/COLLISION-Wave Glider-float.dae" />
+  <xacro:macro name="glider_asv_base" params="namespace debug inertial_reference_frame">
     <!-- Base_link of the model -->
     <link name="${namespace}/base_link">
       <visual>
-        <origin xyz="0 0 0" rpy="0 0 -${0.5*pi}" />
+        <origin xyz="0 0 0" rpy="0 0 ${pi/2}" />
         <geometry>
           <mesh filename="${visual_mesh_file}" scale="1 1 1" />
@@ -37,5 +35,5 @@
       </visual>
       <collision>
-        <origin xyz="0 0 0" rpy="0 0 -${0.5*pi}" />
+        <origin xyz="0 0 0" rpy="0 0 ${pi/2}" />
         <geometry>
           <mesh filename="${collision_mesh_file}" scale="1 1 1" />
@@ -44,87 +42,8 @@
       <inertial>
         <mass value="${mass}"/>
-        <origin xyz="0 0 0" rpy="0 0 0" />
+        <origin xyz="0 0 0" rpy="0 0 ${pi/2}" />
         <inertia ixx="0.3048" ixy="0" ixz="0" iyy="13.976" iyz="0" izz="13.976" />
       </inertial>
     </link>
-    <!-- Dummy propeller plugin properties (rotorConstant = 0) -->
-    <!-- This is for topics used to visualize the propeller roatation  -->
-    <xacro:property name="dummy_plugin_properties_for_visual_rotation">
-      <dynamics>
-        <type>FirstOrder</type>
-        <timeConstant>0.0</timeConstant>
-      </dynamics>
-      <conversion>
-        <type>Basic</type>
-        <rotorConstant>0.0</rotorConstant>
-      </conversion>
-    </xacro:property>
-    <xacro:property name="dummy_link_properties_for_visual_rotation">
-      <xacro:box_inertial x="0" y="0" z="0" mass="0.00001">
-        <origin xyz="0 0 0" rpy="0 0 0"/>
-      </xacro:box_inertial>
-      <collision>
-        <geometry>
-          <cylinder length="0.000001" radius="0.000001"/>
-        </geometry>
-        <origin xyz="0 0 0" rpy="0 0 0"/>
-      </collision>
-    </xacro:property>
-    <!-- First propeller -->
-    <xacro:property name="thruster_id" value="1"/>
-    <joint name="${namespace}/thruster_${thruster_id}_joint" type="continuous">
-      <origin xyz="-0.558 -0.05 0" rpy="0 0 -${0.07*pi}"/>
-      <axis xyz="1 0 0"/>
-      <parent link="${namespace}/base_link"/>
-      <child link="${namespace}/thruster_${thruster_id}"/>
-    </joint>
-    <link name="${namespace}/thruster_${thruster_id}">
-      <xacro:insert_block name="dummy_link_properties_for_visual_rotation"/>
-      <visual>
-        <origin xyz="0.541 0.12 0" rpy="0 0 -${0.46*pi}"/>
-        <geometry>
-          <mesh filename="${right_prop_mesh_file}" scale="1 1 1"/>
-        </geometry>
-      </visual>
-    </link>
-    <gazebo>
-      <plugin name="${namespace}_${thruster_id}_thruster_model" filename="libuuv_thruster_ros_plugin.so">
-        <linkName>${namespace}/thruster_${thruster_id}</linkName>
-        <jointName>${namespace}/thruster_${thruster_id}_joint</jointName>
-        <thrusterID>${thruster_id}</thrusterID>
-        <xacro:insert_block name="dummy_plugin_properties_for_visual_rotation"/>
-      </plugin>
-    </gazebo>
-    <gazebo reference="${namespace}/thruster_${thruster_id}">
-      <selfCollide>false</selfCollide>
-    </gazebo>
-    <!-- Second propeller -->
-    <xacro:property name="thruster_id" value="0"/>
-    <joint name="${namespace}/thruster_${thruster_id}_joint" type="continuous">
-      <origin xyz="-0.558 0.05 0" rpy="0 0 ${0.07*pi+pi}"/>
-      <axis xyz="1 0 0"/>
-      <parent link="${namespace}/base_link"/>
-      <child link="${namespace}/thruster_${thruster_id}"/>
-    </joint>
-    <link name="${namespace}/thruster_${thruster_id}">
-      <xacro:insert_block name="dummy_link_properties_for_visual_rotation"/>
-      <visual>
-        <origin xyz="-0.541 0.12 0" rpy="0 0 ${0.46*pi}"/>
-        <geometry>
-          <mesh filename="${left_prop_mesh_file}" scale="1 1 1"/>
-        </geometry>
-      </visual>
-    </link>
-    <gazebo>
-      <plugin name="${namespace}_${thruster_id}_thruster_model" filename="libuuv_thruster_ros_plugin.so">
-        <linkName>${namespace}/thruster_${thruster_id}</linkName>
-        <jointName>${namespace}/thruster_${thruster_id}_joint</jointName>
-        <thrusterID>${thruster_id}</thrusterID>
-        <xacro:insert_block name="dummy_plugin_properties_for_visual_rotation"/>
-      </plugin>
-    </gazebo>
-    <gazebo reference="${namespace}/thruster_${thruster_id}">
-      <selfCollide>false</selfCollide>
-    </gazebo>
     <!-- Kinematics Plugin -->
     <gazebo>
@@ -137,4 +56,5 @@
         <espg_projection>26987</espg_projection>
         <!-- Kinematics coefficients -->
+        <surface_vehicle>true</surface_vehicle>
         <f_pitch_battpos_cal_m>1.2565</f_pitch_battpos_cal_m>
         <f_pitch_battpos_cal_b>-0.055</f_pitch_battpos_cal_b>
@@ -192,5 +112,5 @@
       voltage="4.2"
       update_rate="2.0"/>
-    <xacro:include filename="$(find glider_hybrid_whoi_description)/urdf/glider_hybrid_whoi_sensors_kinematics.xacro"/>
+    <xacro:include filename="$(find glider_hybrid_whoi_description)/urdf/glider_asv_sensors_kinematics.xacro"/>
   </xacro:macro>
 </robot>
