Commit message: add altimeter using simple dvl sensor

File: glider_hybrid_whoi_description/urdf/glider_hybrid_whoi_sensors_kinematics.xacro (robot description, xacro)
@@ -23,28 +23,16 @@
       suffix=""
       parent_link="${namespace}/base_link"
-      topic="dvl"
+      topic="altimeter"
       scale="0.62"
       noise_sigma="0"
       noise_amplitude="0"
-      update_rate="7"
+      update_rate="0.25"
       reference_frame="world">
-      <origin xyz="0.0 0.0 -0.0825" rpy="0 ${0.5*pi} 0" />
+      <origin xyz="0.0 0.0 -0.0825" rpy="0 ${0.355556*pi} 0" />
     </xacro:dvl_plugin_macro>
-    <xacro:switchable_battery_consumer_macro
-      link_name="${namespace}/dvl_link"
-      battery_link="${namespace}/battery_link"
-      battery_name="${namespace}/battery"
-      power_load="25"
-      topic="${namespace}/dvl/state"/>
     <!-- IMU  -->
     <xacro:default_imu namespace="${namespace}" parent_link="${namespace}/base_link">
       <origin xyz="0 0 0" rpy="0 0 0"/>
     </xacro:default_imu>
-    <xacro:switchable_battery_consumer_macro
-      link_name="${namespace}/imu_link"
-      battery_link="${namespace}/battery_link"
-      battery_name="${namespace}/battery"
-      power_load="20"
-      topic="${namespace}/imu/state"/>
     <!-- Mount a camera -->
     <xacro:regular_camera_plugin_macro
@@ -65,9 +53,9 @@
     <!-- Mount a GPS. -->
     <xacro:default_gps namespace="${namespace}" parent_link="${namespace}/base_link" />
-    <xacro:switchable_battery_consumer_macro
+    <!-- <xacro:switchable_battery_consumer_macro
       link_name="${namespace}/gps_link"
       battery_link="${namespace}/battery_link"
       battery_name="${namespace}/battery"
       power_load="5"
-      topic=""/>
+      topic=""/> -->
 </robot>

Commit message: add depth/pressure sensor

File: glider_hybrid_whoi_description/urdf/glider_hybrid_whoi_sensors_kinematics.xacro (robot description, xacro)
@@ -37,4 +37,20 @@
       power_load="25"
       topic="${namespace}/dvl/state"/>
+    <xacro:pressure_plugin_macro
+      namespace="${namespace}"
+      suffix=""
+      parent_link="${namespace}/base_link"
+      topic="pressure"
+      mass="0.015"
+      update_rate="10"
+      range="1362"
+      noise_sigma="3.0"
+      noise_amplitude="0.0"
+      estimateDepth="true"
+      standardPressure="101.325"
+      kPaPerM="9.80638">
+      <inertia ixx="0.00001" ixy="0.0" ixz="0.0" iyy="0.00001" iyz="0.0" izz="0.00001" />
+      <origin xyz="0.0 0.0 -0.0825" rpy="0 ${0.5*pi} 0" />
+    </xacro:pressure_plugin_macro>
     <!-- IMU  -->
     <xacro:default_imu namespace="${namespace}" parent_link="${namespace}/base_link">

Commit message: add pressure sensor

File: glider_hybrid_whoi_description/urdf/glider_hybrid_whoi_sensors_kinematics.xacro (robot description, xacro)
@@ -18,26 +18,25 @@
       parent_link="${namespace}/base_link"
       inertial_reference_frame="${inertial_reference_frame}" />
-    <!-- DVL sensor -->
-    <!-- <xacro:dvl_plugin_macro
+    <xacro:include filename="$(find nps_uw_sensors_gazebo)/urdf/whoi_teledyne_whn_beams.xacro"/>
+    <xacro:teledyne_whn_macro
+      name="dvl" namespace="dvl" xyz="0 0 0"
+      dvl_topic="dvl" ranges_topic="ranges"
+      robot_link="${namespace}/base_link" joint_xyz="0 0 0" scale="0.25 0.25 0.25" ray_visual="1"/>
+    <xacro:pressure_plugin_macro
       namespace="${namespace}"
       suffix=""
       parent_link="${namespace}/base_link"
-      topic="altimeter"
-      scale="0.62"
-      noise_sigma="0"
-      noise_amplitude="0"
-      update_rate="0.25"
-      reference_frame="world">
+      topic="pressure"
+      mass="0.015"
+      update_rate="10"
+      range="1362"
+      noise_sigma="3.0"
+      noise_amplitude="0.0"
+      estimateDepth="true"
+      standardPressure="101.325"
+      kPaPerM="9.80638">
+      <inertia ixx="0.00001" ixy="0.0" ixz="0.0" iyy="0.00001" iyz="0.0" izz="0.00001" />
       <origin xyz="0.0 0.0 -0.0825" rpy="0 ${0.5*pi} 0" />
-    </xacro:dvl_plugin_macro> -->
-  <xacro:include filename="$(find nps_uw_sensors_gazebo)/urdf/whoi_teledyne_whn_beams.xacro"/>
-  <xacro:teledyne_whn_macro
-    name="dvl" namespace="dvl" xyz="0 0 0"
-    dvl_topic="dvl" ranges_topic="ranges"
-    robot_link="${namespace}/base_link" joint_xyz="0 0 0" scale="0.25 0.25 0.25" ray_visual="1"/>
-    <!-- IMU  -->
-    <xacro:default_imu namespace="${namespace}" parent_link="${namespace}/base_link">
-      <origin xyz="0 0 0" rpy="0 0 0"/>
-    </xacro:default_imu>
+    </xacro:pressure_plugin_macro>
     <!-- Hector IMU -->
     <xacro:include filename="$(find glider_hybrid_whoi_description)/urdf/uw_hector_imu_plugin.xacro"/>
@@ -66,9 +65,3 @@
     <!-- Hector GPS -->
     <xacro:include filename="$(find glider_hybrid_whoi_description)/urdf/uw_hector_gps_plugin.xacro"/>
-    <!-- <xacro:switchable_battery_consumer_macro
-      link_name="${namespace}/gps_link"
-      battery_link="${namespace}/battery_link"
-      battery_name="${namespace}/battery"
-      power_load="5"
-      topic=""/> -->
 </robot>

Commit message: add back altimeter sensor using dvl plugin. Topic is published as altimeter

File: glider_hybrid_whoi_description/urdf/glider_hybrid_whoi_sensors_kinematics.xacro (robot description, xacro)
@@ -18,4 +18,5 @@
       parent_link="${namespace}/base_link"
       inertial_reference_frame="${inertial_reference_frame}" />
+    <!-- DVL -->
     <xacro:include filename="$(find nps_uw_sensors_gazebo)/urdf/whoi_teledyne_whn_beams.xacro"/>
     <xacro:teledyne_whn_macro
@@ -23,4 +24,18 @@
       dvl_topic="dvl" ranges_topic="ranges"
       robot_link="${namespace}/base_link" joint_xyz="0 0 0" scale="0.25 0.25 0.25" ray_visual="1"/>
+    <!-- Altimeter -->
+    <xacro:dvl_plugin_macro
+      namespace="${namespace}"
+      suffix=""
+      parent_link="${namespace}/base_link"
+      topic="altimeter"
+      scale="0.62"
+      noise_sigma="0"
+      noise_amplitude="0"
+      update_rate="0.25"
+      reference_frame="world">
+      <origin xyz="0.0 0.0 -0.0825" rpy="0 ${0.355556*pi} 0" />
+    </xacro:dvl_plugin_macro>
+    <!-- Pressure  -->
     <xacro:pressure_plugin_macro
       namespace="${namespace}"

Commit message: fix pressure sensor location

File: glider_hybrid_whoi_description/urdf/glider_hybrid_whoi_sensors_kinematics.xacro (robot description, xacro)
@@ -52,5 +52,5 @@
       kPaPerM="9.80638">
       <inertia ixx="0.00001" ixy="0.0" ixz="0.0" iyy="0.00001" iyz="0.0" izz="0.00001" />
-      <origin xyz="0.0 0.0 -0.0825" rpy="0 ${0.5*pi} 0" />
+      <origin xyz="0.0 0.0 0.0" rpy="0 ${0.355556*pi} 0" />
     </xacro:pressure_plugin_macro>
     <!-- Hector IMU -->
