Commit message: Commanding function ready

File: glider_hybrid_whoi_description/urdf/glider_hybrid_whoi_base_kinematics.xacro (robot description, xacro)
@@ -19,6 +19,6 @@
   <xacro:include filename="$(find uuv_gazebo_ros_plugins)/urdf/snippets.xacro"/>
   <!-- Properties -->
-  <xacro:property name="mass" value="56.0"/>
-  <xacro:property name="hull_mass" value="48.2"/>
+  <xacro:property name="mass" value="1000.0"/>
+  <!-- <xacro:property name="hull_mass" value="48.2"/>
   <xacro:property name="shifter_mass" value="7.8"/>
   <xacro:property name="length" value="2.0"/>
@@ -31,22 +31,20 @@
   <xacro:property name="max_mass_pos" value="0.03"/>
   <xacro:property name="max_ballast_vol" value="2.4e-04"/>
-  <xacro:property name="volume" value="99999999"/> <!-- usage? Neutural buoyancy disabled using zero gravity world-->
+  <xacro:property name="volume" value="99999999"/>
   <xacro:property name="cob" value="0 0 0"/>
   <xacro:property name="cog" value="0 0 0.0054"/>
-  <xacro:property name="rho" value="1024.0"/>
-  <!-- <xacro:property name="visual_mesh_file" value="file://$(find glider_hybrid_whoi_description)/mesh/glider_hybrid_whoi.dae"/>
-  <xacro:property name="collision_mesh_file" value="file://$(find glider_hybrid_whoi_description)/mesh/glider_hybrid_whoi_collision.dae"/>
-  <xacro:property name="prop_mesh_file" value="file://$(find glider_hybrid_whoi_description)/mesh/glider_hybrid_whoi_propeller.dae"/>
-  <xacro:property name="fin_mesh_file" value="file://$(find glider_hybrid_whoi_description)/mesh/glider_hybrid_whoi_fin.dae"/> -->
-  <xacro:property name="visual_mesh_file" value="file://$(find glider_hybrid_whoi_description)/mesh/eca_a9/eca_a9.dae"/>
+  <xacro:property name="rho" value="1024.0"/> -->
+  <xacro:property name="visual_mesh_file" value="file://$(find uuv_dave)/models/glider_hybrid_whoi/mesh/glider_hybrid_whoi_body.dae" />
+  <xacro:property name="collision_mesh_file" value="file://$(find uuv_dave)/models/glider_hybrid_whoi/mesh/glider_hybrid_whoi_collision.dae" />
+  <xacro:property name="left_prop_mesh_file" value="file://$(find uuv_dave)/models/glider_hybrid_whoi/mesh/glider_hybrid_whoi_left_propeller.dae" />
+  <xacro:property name="right_prop_mesh_file" value="file://$(find uuv_dave)/models/glider_hybrid_whoi/mesh/glider_hybrid_whoi_right_propeller.dae" />
+  <!-- <xacro:property name="visual_mesh_file" value="file://$(find glider_hybrid_whoi_description)/mesh/eca_a9/eca_a9.dae"/>
   <xacro:property name="collision_mesh_file" value="file://$(find glider_hybrid_whoi_description)/mesh/eca_a9/eca_a9.stl"/>
   <xacro:property name="prop_mesh_file" value="file://$(find glider_hybrid_whoi_description)/mesh/eca_a9/eca_a9_propeller.dae"/>
-  <xacro:property name="fin_mesh_file" value="file://$(find glider_hybrid_whoi_description)/mesh/eca_a9/eca_a9_fin.dae"/>
+  <xacro:property name="fin_mesh_file" value="file://$(find glider_hybrid_whoi_description)/mesh/eca_a9/eca_a9_fin.dae"/> -->
   <xacro:macro name="glider_hybrid_whoi_base" params="namespace debug inertial_reference_frame">
-    <!-- <link name="dummy">
-    </link> -->
     <link name="${namespace}/base_link">
       <visual>
-        <origin xyz="0 0 0" rpy="0 0 0"/>
+        <origin xyz="0 0 0" rpy="0 0 -1.5708" />
         <geometry>
           <mesh filename="${visual_mesh_file}" scale="1 1 1" />
@@ -54,23 +52,54 @@
       </visual>
       <collision>
-        <origin xyz="0 0 0" rpy="0 0 0"/>
+        <origin xyz="0 0 0" rpy="0 0 -1.5708" />
         <geometry>
           <mesh filename="${collision_mesh_file}" scale="1 1 1" />
         </geometry>
       </collision>
-      <!-- This inertial input is dummy input. The values will be changed within glider kinamatics plugin with Fossen's-->
       <inertial>
-        <origin xyz="0 0 0" rpy="0 0 0"/>
-        <mass value="${mass}" />
-        <inertia ixx="0.3048" ixy="0" ixz="0"
-                 iyy="13.9760" iyz="0"
-                 izz="13.9760" />
+        <mass value="${mass}"/>
+        <origin xyz="0 0 0" rpy="0 0 0" />
+        <inertia ixx="30.0" ixy="0" ixz="0" iyy="0.6" iyz="0" izz="5.0" />
       </inertial>
     </link>
-    <!-- Dummy joint to fix inertial definition at urdf warnings -->
-    <!-- <joint name="dummy_joint" type="fixed">
-      <parent link="dummy"/>
-      <child link="${namespace}/base_link"/>
-    </joint> -->
+    <link name="${namespace}/left_propeller_link">
+      <visual>
+        <origin xyz="0 0 0" rpy="0 0 0 " />
+        <geometry>
+          <mesh filename="${left_prop_mesh_file}" scale="1 1 1" />
+        </geometry>
+      </visual>
+    </link>
+    <joint name="${namespace}/left_propeller_joint" type="continuous">
+      <origin xyz="0 0 0" rpy="0 0 0" />
+      <parent link="${namespace}/base_link"/>
+      <child link="${namespace}/left_propeller_link"/>
+      <axis xyz="0 1 0" />
+    </joint>
+    <link name="${namespace}/right_propeller_link">
+      <visual>
+        <origin xyz="0 0 0" rpy="0 0 0" />
+        <geometry>
+          <mesh filename="${right_prop_mesh_file}" scale="1 1 1" />
+        </geometry>
+      </visual>
+    </link>
+    <joint name="${namespace}/right_propeller_joint" type="continuous">
+      <origin xyz="0 0 0" rpy="0 0 0" />
+      <parent link="${namespace}/base_link"/>
+      <child link="${namespace}/right_propeller_link"/>
+      <axis xyz="0 1 0" />
+    </joint>
+    <link name='${namespace}/battery_link2'>
+      <origin xyz="0 0 0" rpy="0 0 0" />
+      <battery name='${namespace}/battery'>
+        <voltage>4.2</voltage>
+      </battery>
+    </link>
+    <joint name='${namespace}/battery_joint2' type='fixed'>
+      <origin xyz="0 0 0" rpy="0 0 0" />
+      <parent link="${namespace}/base_link"/>
+      <child link="${namespace}/battery_link2"/>
+    </joint>
     <!-- Set up hydrodynamic plugin -->
     <gazebo>

Commit message: Added DVL sensor and new worlds for altitude status

File: glider_hybrid_whoi_description/urdf/glider_hybrid_whoi_base_kinematics.xacro (robot description, xacro)
@@ -20,31 +20,12 @@
   <!-- Properties -->
   <xacro:property name="mass" value="1000.0"/>
-  <!-- <xacro:property name="hull_mass" value="48.2"/>
-  <xacro:property name="shifter_mass" value="7.8"/>
-  <xacro:property name="length" value="2.0"/>
-  <xacro:property name="radius" value="0.105"/>
-  <xacro:property name="diameter" value="${radius*2}"/>
-  <xacro:property name="area" value="${radius*radius*3.141592}"/>
-  <xacro:property name="ballast_tank_radius" value="0.07"/>
-  <xacro:property name="initial_mass_pos" value="0.4"/>
-  <xacro:property name="initial_ballast_pos" value="0.711"/>
-  <xacro:property name="max_mass_pos" value="0.03"/>
-  <xacro:property name="max_ballast_vol" value="2.4e-04"/>
-  <xacro:property name="volume" value="99999999"/>
-  <xacro:property name="cob" value="0 0 0"/>
-  <xacro:property name="cog" value="0 0 0.0054"/>
-  <xacro:property name="rho" value="1024.0"/> -->
   <xacro:property name="visual_mesh_file" value="file://$(find uuv_dave)/models/glider_hybrid_whoi/mesh/glider_hybrid_whoi_body.dae" />
   <xacro:property name="collision_mesh_file" value="file://$(find uuv_dave)/models/glider_hybrid_whoi/mesh/glider_hybrid_whoi_collision.dae" />
   <xacro:property name="left_prop_mesh_file" value="file://$(find uuv_dave)/models/glider_hybrid_whoi/mesh/glider_hybrid_whoi_left_propeller.dae" />
   <xacro:property name="right_prop_mesh_file" value="file://$(find uuv_dave)/models/glider_hybrid_whoi/mesh/glider_hybrid_whoi_right_propeller.dae" />
-  <!-- <xacro:property name="visual_mesh_file" value="file://$(find glider_hybrid_whoi_description)/mesh/eca_a9/eca_a9.dae"/>
-  <xacro:property name="collision_mesh_file" value="file://$(find glider_hybrid_whoi_description)/mesh/eca_a9/eca_a9.stl"/>
-  <xacro:property name="prop_mesh_file" value="file://$(find glider_hybrid_whoi_description)/mesh/eca_a9/eca_a9_propeller.dae"/>
-  <xacro:property name="fin_mesh_file" value="file://$(find glider_hybrid_whoi_description)/mesh/eca_a9/eca_a9_fin.dae"/> -->
   <xacro:macro name="glider_hybrid_whoi_base" params="namespace debug inertial_reference_frame">
     <link name="${namespace}/base_link">
       <visual>
-        <origin xyz="0 0 0" rpy="0 0 -1.5708" />
+        <origin xyz="0 0 0" rpy="0 0 -${0.5*pi}" />
         <geometry>
           <mesh filename="${visual_mesh_file}" scale="1 1 1" />
@@ -52,5 +33,5 @@
       </visual>
       <collision>
-        <origin xyz="0 0 0" rpy="0 0 -1.5708" />
+        <origin xyz="0 0 0" rpy="0 0 -${0.5*pi}" />
         <geometry>
           <mesh filename="${collision_mesh_file}" scale="1 1 1" />
@@ -65,5 +46,5 @@
     <link name="${namespace}/left_propeller_link">
       <visual>
-        <origin xyz="0 0 0" rpy="0 0 0 " />
+        <origin xyz="0 0 0" rpy="0 0 -${0.25*pi}" />
         <geometry>
           <mesh filename="${left_prop_mesh_file}" scale="1 1 1" />
@@ -71,6 +52,6 @@
       </visual>
     </link>
-    <joint name="${namespace}/left_propeller_joint" type="continuous">
-      <origin xyz="0 0 0" rpy="0 0 0" />
+    <joint name="${namespace}/left_propeller_joint" type="fixed">
+      <origin xyz="0 0 0" rpy="0 0 -${0.25*pi}" />
       <parent link="${namespace}/base_link"/>
       <child link="${namespace}/left_propeller_link"/>
@@ -79,5 +60,5 @@
     <link name="${namespace}/right_propeller_link">
       <visual>
-        <origin xyz="0 0 0" rpy="0 0 0" />
+        <origin xyz="0 0 0" rpy="0 0 -${0.25*pi}" />
         <geometry>
           <mesh filename="${right_prop_mesh_file}" scale="1 1 1" />
@@ -85,20 +66,9 @@
       </visual>
     </link>
-    <joint name="${namespace}/right_propeller_joint" type="continuous">
-      <origin xyz="0 0 0" rpy="0 0 0" />
+    <joint name="${namespace}/right_propeller_joint" type="fixed">
+      <origin xyz="0 0 0" rpy="0 0 -${0.25*pi}" />
       <parent link="${namespace}/base_link"/>
       <child link="${namespace}/right_propeller_link"/>
       <axis xyz="0 1 0" />
-    </joint>
-    <link name='${namespace}/battery_link2'>
-      <origin xyz="0 0 0" rpy="0 0 0" />
-      <battery name='${namespace}/battery'>
-        <voltage>4.2</voltage>
-      </battery>
-    </link>
-    <joint name='${namespace}/battery_joint2' type='fixed'>
-      <origin xyz="0 0 0" rpy="0 0 0" />
-      <parent link="${namespace}/base_link"/>
-      <child link="${namespace}/battery_link2"/>
     </joint>
     <!-- Set up hydrodynamic plugin -->
@@ -108,71 +78,7 @@
         <writeLog>1</writeLog>
       </plugin>
-      <!-- <plugin name="${namespace}_hybrid_glider_plugin" filename="libhybrid_glider_underwater_object_ros_plugin.so">
-        <fluid_density>${rho}</fluid_density>
-        <flow_velocity_topic>hydrodynamics/current_velocity</flow_velocity_topic>
-        <debug>${debug}</debug>
-        <writeLog>1</writeLog>
-        <link name="${namespace}/base_link">
-          <volume>${volume}</volume>
-          <center_of_buoyancy>${cob}</center_of_buoyancy>
-          <center_of_gravity>${cog}</center_of_gravity>
-          <neutrally_buoyant>0</neutrally_buoyant>
-          <hard_code_input>0</hard_code_input>
-          <hydrodynamic_model>
-            <type>fossen</type>
-            <added_mass>
-              100 0   0   0   0   0
-              0   100 0   0   0   0
-              0   0   100 0   0   0
-              0   0   0   100 0   0
-              0   0   0   0   100 0
-              0   0   0   0   0   100
-            </added_mass>
-            <linear_damping>
-              0       0       0       0       0       0
-              0       0       0       0       0       0
-              0       0       -14     0       0       0
-              0       0       0       0       0       0
-              0       0       0       0       -12     0
-              0       0       0       0       0       0
-            </linear_damping>
-          </hydrodynamic_model>
-            <ballast_radius>${ballast_tank_radius}</ballast_radius>
-            <hull_length>${length}</hull_length>
-            <hull_radius>${radius}</hull_radius>
-            <hull_mass>${hull_mass}</hull_mass>
-            <shifter_mass>${shifter_mass}</shifter_mass>
-            <initial_mass_position>${initial_mass_pos}</initial_mass_position>
-            <initial_ballast_position>${initial_ballast_pos}</initial_ballast_position>
-            <max_mass_position>${max_mass_pos}</max_mass_position>
-            <max_ballast_volume>${max_ballast_vol}</max_ballast_volume>
-        </link>
-      </plugin> -->
     </gazebo>
-    <!-- Instantiate Fins -->
-    <!-- <xacro:fin_macro namespace="${namespace}" fin_id="0">
-      <origin xyz="-0.70777 -0.07876 0.078586" rpy="0.7904 -0.0998 -0.1003" />
-    </xacro:fin_macro>
-    <xacro:fin_macro namespace="${namespace}" fin_id="1">
-      <origin xyz="-0.70777 -0.07876 -0.078586" rpy="2.3512 0.0998 -0.1003" />
-    </xacro:fin_macro> -->
-    <!--
-    <xacro:fin_macro namespace="${namespace}" fin_id="2">
-      <origin xyz="-0.70777 0.07876 -0.078586" rpy="-2.3512 0.0998 0.1003" />
-    </xacro:fin_macro>
-    <xacro:fin_macro namespace="${namespace}" fin_id="3">
-      <origin xyz="-0.70777 0.07876 0.078586" rpy="-0.7904 -0.0998 0.1003" />
-    </xacro:fin_macro>
-    -->
-    <!-- <xacro:thruster_module_first_order_basic_fcn_macro
-      namespace="${namespace}"
-      thruster_id="0"
-      mesh_filename="${prop_mesh_file}"
-      dyn_time_constant="0.1"
-      rotor_constant="0.00049">
-      <origin xyz="-0.9676 0 0" rpy="0 0 ${pi}" />
-    </xacro:thruster_module_first_order_basic_fcn_macro> -->
     <!-- TODO: Parametrize the battery unit -->
-    <!-- <xacro:basic_linear_battery_macro
+    <xacro:basic_linear_battery_macro
       namespace="${namespace}"
       parent_link="${namespace}/base_link"
@@ -185,6 +91,6 @@
       smooth_current_tau="1.9499"
       voltage="4.2"
-      update_rate="2.0"/> -->
-    <xacro:include filename="$(find glider_hybrid_whoi_description)/urdf/glider_hybrid_whoi_sensors_test.xacro"/>
+      update_rate="2.0"/>
+    <xacro:include filename="$(find glider_hybrid_whoi_description)/urdf/glider_hybrid_whoi_sensors_kinematics.xacro"/>
   </xacro:macro>
 </robot>

File: glider_hybrid_whoi_description/urdf/glider_hybrid_whoi_base_test.xacro (robot description, xacro)
@@ -35,18 +35,12 @@
   <xacro:property name="cog" value="0 0 0.0054"/>
   <xacro:property name="rho" value="1024.0"/>
-  <!-- <xacro:property name="visual_mesh_file" value="file://$(find glider_hybrid_whoi_description)/mesh/glider_hybrid_whoi.dae"/>
-  <xacro:property name="collision_mesh_file" value="file://$(find glider_hybrid_whoi_description)/mesh/glider_hybrid_whoi_collision.dae"/>
-  <xacro:property name="prop_mesh_file" value="file://$(find glider_hybrid_whoi_description)/mesh/glider_hybrid_whoi_propeller.dae"/>
-  <xacro:property name="fin_mesh_file" value="file://$(find glider_hybrid_whoi_description)/mesh/glider_hybrid_whoi_fin.dae"/> -->
-  <xacro:property name="visual_mesh_file" value="file://$(find glider_hybrid_whoi_description)/mesh/eca_a9/eca_a9.dae"/>
-  <xacro:property name="collision_mesh_file" value="file://$(find glider_hybrid_whoi_description)/mesh/eca_a9/eca_a9.stl"/>
-  <xacro:property name="prop_mesh_file" value="file://$(find glider_hybrid_whoi_description)/mesh/eca_a9/eca_a9_propeller.dae"/>
-  <xacro:property name="fin_mesh_file" value="file://$(find glider_hybrid_whoi_description)/mesh/eca_a9/eca_a9_fin.dae"/>
+  <xacro:property name="visual_mesh_file" value="file://$(find uuv_dave)/models/glider_hybrid_whoi/mesh/glider_hybrid_whoi_body.dae" />
+  <xacro:property name="collision_mesh_file" value="file://$(find uuv_dave)/models/glider_hybrid_whoi/mesh/glider_hybrid_whoi_collision.dae" />
+  <xacro:property name="left_prop_mesh_file" value="file://$(find uuv_dave)/models/glider_hybrid_whoi/mesh/glider_hybrid_whoi_left_propeller.dae" />
+  <xacro:property name="right_prop_mesh_file" value="file://$(find uuv_dave)/models/glider_hybrid_whoi/mesh/glider_hybrid_whoi_right_propeller.dae" />
   <xacro:macro name="glider_hybrid_whoi_base" params="namespace debug inertial_reference_frame">
-    <!-- <link name="dummy">
-    </link> -->
     <link name="${namespace}/base_link">
       <visual>
-        <origin xyz="0 0 0" rpy="0 0 0"/>
+        <origin xyz="0 0 0" rpy="0 0 -1.5708" />
         <geometry>
           <mesh filename="${visual_mesh_file}" scale="1 1 1" />
@@ -54,23 +48,54 @@
       </visual>
       <collision>
-        <origin xyz="0 0 0" rpy="0 0 0"/>
+        <origin xyz="0 0 0" rpy="0 0 -1.5708" />
         <geometry>
           <mesh filename="${collision_mesh_file}" scale="1 1 1" />
         </geometry>
       </collision>
-      <!-- This inertial input is dummy input. The values will be changed within glider kinamatics plugin with Fossen's-->
       <inertial>
-        <origin xyz="0 0 0" rpy="0 0 0"/>
-        <mass value="${mass}" />
-        <inertia ixx="0.3048" ixy="0" ixz="0"
-                 iyy="13.9760" iyz="0"
-                 izz="13.9760" />
+        <mass value="${mass}"/>
+        <origin xyz="0 0 0" rpy="0 0 0" />
+        <inertia ixx="0.3048" ixy="0" ixz="0" iyy="13.976" iyz="0" izz="13.976" />
       </inertial>
     </link>
-    <!-- Dummy joint to fix inertial definition at urdf warnings -->
-    <!-- <joint name="dummy_joint" type="fixed">
-      <parent link="dummy"/>
-      <child link="${namespace}/base_link"/>
-    </joint> -->
+    <link name="${namespace}/left_propeller_link">
+      <visual>
+        <origin xyz="0 0 0" rpy="0 0 0 " />
+        <geometry>
+          <mesh filename="${left_prop_mesh_file}" scale="1 1 1" />
+        </geometry>
+      </visual>
+    </link>
+    <joint name="${namespace}/left_propeller_joint" type="continuous">
+      <origin xyz="0 0 0" rpy="0 0 0" />
+      <parent link="${namespace}/base_link"/>
+      <child link="${namespace}/left_propeller_link"/>
+      <axis xyz="0 1 0" />
+    </joint>
+    <link name="${namespace}/right_propeller_link">
+      <visual>
+        <origin xyz="0 0 0" rpy="0 0 0" />
+        <geometry>
+          <mesh filename="${right_prop_mesh_file}" scale="1 1 1" />
+        </geometry>
+      </visual>
+    </link>
+    <joint name="${namespace}/right_propeller_joint" type="continuous">
+      <origin xyz="0 0 0" rpy="0 0 0" />
+      <parent link="${namespace}/base_link"/>
+      <child link="${namespace}/right_propeller_link"/>
+      <axis xyz="0 1 0" />
+    </joint>
+    <link name='${namespace}/battery_link2'>
+      <origin xyz="0 0 0" rpy="0 0 0" />
+      <battery name='${namespace}/battery'>
+        <voltage>4.2</voltage>
+      </battery>
+    </link>
+    <joint name='${namespace}/battery_joint2' type='fixed'>
+      <origin xyz="0 0 0" rpy="0 0 0" />
+      <parent link="${namespace}/base_link"/>
+      <child link="${namespace}/battery_link2"/>
+    </joint>
     <!-- Set up hydrodynamic plugin -->
     <gazebo>
@@ -96,12 +121,4 @@
               0   0   0   0   0   100
             </added_mass>
-            <!-- <linear_damping_forward_speed>
-              0       0       0       0       0       0
-              0       0       0       0       0       0
-              0       0       -14     0       0       0
-              0       0       0       0       0       0
-              0       0       0       0       -12     0
-              0       0       0       0       0       0
-            </linear_damping_forward_speed> -->
             <linear_damping>
               0       0       0       0       0       0

File: glider_hybrid_whoi_description/urdf/glider_hybrid_whoi_sensors_test.xacro (robot description, xacro)
@@ -29,5 +29,5 @@
       update_rate="7"
       reference_frame="world">
-      <origin xyz="0.4785 0.0 -0.0825" rpy="0 ${0.5*pi} 0" />
+      <origin xyz="0.0 0.0 -0.0825" rpy="0 0 -${0.5*pi}" />
     </xacro:dvl_plugin_macro>
     <xacro:switchable_battery_consumer_macro
