Commit message: visual effects for propeller rotation added

File: glider_hybrid_whoi_description/urdf/glider_hybrid_whoi_base_kinematics.xacro (robot description, xacro)
@@ -19,9 +19,9 @@
   <xacro:include filename="$(find uuv_gazebo_ros_plugins)/urdf/snippets.xacro"/>
   <!-- Properties -->
-  <xacro:property name="mass" value="1000.0"/>
-  <xacro:property name="visual_mesh_file" value="file://$(find uuv_dave)/models/glider_hybrid_whoi/mesh/glider_hybrid_whoi_body.dae" />
-  <xacro:property name="collision_mesh_file" value="file://$(find uuv_dave)/models/glider_hybrid_whoi/mesh/glider_hybrid_whoi_collision.dae" />
-  <xacro:property name="left_prop_mesh_file" value="file://$(find uuv_dave)/models/glider_hybrid_whoi/mesh/glider_hybrid_whoi_left_propeller.dae" />
-  <xacro:property name="right_prop_mesh_file" value="file://$(find uuv_dave)/models/glider_hybrid_whoi/mesh/glider_hybrid_whoi_right_propeller.dae" />
+  <xacro:property name="mass" value="10000.0"/>
+  <xacro:property name="visual_mesh_file" value="file://$(find glider_hybrid_whoi_description)/mesh/glider_hybrid_whoi/glider_hybrid_whoi_body.dae" />
+  <xacro:property name="collision_mesh_file" value="file://$(find glider_hybrid_whoi_description)/mesh/glider_hybrid_whoi/glider_hybrid_whoi_collision.dae" />
+  <xacro:property name="left_prop_mesh_file" value="file://$(find glider_hybrid_whoi_description)/mesh/glider_hybrid_whoi/glider_hybrid_whoi_left_propeller.dae" />
+  <xacro:property name="right_prop_mesh_file" value="file://$(find glider_hybrid_whoi_description)/mesh/glider_hybrid_whoi/glider_hybrid_whoi_right_propeller.dae" />
   <xacro:macro name="glider_hybrid_whoi_base" params="namespace debug inertial_reference_frame">
     <link name="${namespace}/base_link">
@@ -44,32 +44,88 @@
       </inertial>
     </link>
-    <link name="${namespace}/left_propeller_link">
+  <xacro:property name="thruster_id" value="1"/>
+    <joint name="${namespace}/thruster_${thruster_id}_joint" type="continuous">
+      <origin xyz="-0.558 -0.05 0" rpy="0 0 -${0.07*pi}"/>
+      <axis xyz="1 0 0"/>
+      <parent link="${namespace}/base_link"/>
+      <child link="${namespace}/thruster_${thruster_id}"/>
+    </joint>
+    <link name="${namespace}/thruster_${thruster_id}">
+      <xacro:box_inertial x="0" y="0" z="0" mass="0.00001">
+        <origin xyz="0 0 0" rpy="0 0 0"/>
+      </xacro:box_inertial>
       <visual>
-        <origin xyz="0 0 0" rpy="0 0 -${0.25*pi}" />
+        <origin xyz="0.541 0.12 0" rpy="0 0 -${0.46*pi}"/>
         <geometry>
-          <mesh filename="${left_prop_mesh_file}" scale="1 1 1" />
+          <mesh filename="${right_prop_mesh_file}" scale="1 1 1"/>
         </geometry>
       </visual>
+      <collision>
+        <geometry>
+          <cylinder length="0.000001" radius="0.000001"/>
+        </geometry>
+        <origin xyz="0 0 0" rpy="0 0 0"/>
+      </collision>
     </link>
-    <joint name="${namespace}/left_propeller_joint" type="fixed">
-      <origin xyz="0 0 0" rpy="0 0 -${0.25*pi}" />
+    <gazebo>
+      <plugin name="${namespace}_${thruster_id}_thruster_model" filename="libuuv_thruster_ros_plugin.so">
+        <linkName>${namespace}/thruster_${thruster_id}</linkName>
+        <jointName>${namespace}/thruster_${thruster_id}_joint</jointName>
+        <thrusterID>${thruster_id}</thrusterID>
+        <dynamics>
+          <type>FirstOrder</type>
+          <timeConstant>0.0</timeConstant>
+        </dynamics>
+        <conversion>
+          <type>Basic</type>
+          <rotorConstant>0.0</rotorConstant>
+        </conversion>
+      </plugin>
+    </gazebo>
+    <gazebo reference="${namespace}/thruster_${thruster_id}">
+      <selfCollide>false</selfCollide>
+    </gazebo>
+    <xacro:property name="thruster_id" value="0"/>
+    <joint name="${namespace}/thruster_${thruster_id}_joint" type="continuous">
+      <origin xyz="-0.558 0.05 0" rpy="0 0 ${0.07*pi+pi}"/>
+      <axis xyz="1 0 0"/>
       <parent link="${namespace}/base_link"/>
-      <child link="${namespace}/left_propeller_link"/>
-      <axis xyz="0 1 0" />
+      <child link="${namespace}/thruster_${thruster_id}"/>
     </joint>
-    <link name="${namespace}/right_propeller_link">
+    <link name="${namespace}/thruster_${thruster_id}">
+      <xacro:box_inertial x="0" y="0" z="0" mass="0.00001">
+        <origin xyz="0 0 0" rpy="0 0 0"/>
+      </xacro:box_inertial>
       <visual>
-        <origin xyz="0 0 0" rpy="0 0 -${0.25*pi}" />
+        <origin xyz="-0.541 0.12 0" rpy="0 0 ${0.46*pi}"/>
         <geometry>
-          <mesh filename="${right_prop_mesh_file}" scale="1 1 1" />
+          <mesh filename="${left_prop_mesh_file}" scale="1 1 1"/>
         </geometry>
       </visual>
+      <collision>
+        <geometry>
+          <cylinder length="0.000001" radius="0.000001"/>
+        </geometry>
+        <origin xyz="0 0 0" rpy="0 0 0"/>
+      </collision>
     </link>
-    <joint name="${namespace}/right_propeller_joint" type="fixed">
-      <origin xyz="0 0 0" rpy="0 0 -${0.25*pi}" />
-      <parent link="${namespace}/base_link"/>
-      <child link="${namespace}/right_propeller_link"/>
-      <axis xyz="0 1 0" />
-    </joint>
+    <gazebo>
+      <plugin name="${namespace}_${thruster_id}_thruster_model" filename="libuuv_thruster_ros_plugin.so">
+        <linkName>${namespace}/thruster_${thruster_id}</linkName>
+        <jointName>${namespace}/thruster_${thruster_id}_joint</jointName>
+        <thrusterID>${thruster_id}</thrusterID>
+        <dynamics>
+          <type>FirstOrder</type>
+          <timeConstant>0.0</timeConstant>
+        </dynamics>
+        <conversion>
+          <type>Basic</type>
+          <rotorConstant>0.0</rotorConstant>
+        </conversion>
+      </plugin>
+    </gazebo>
+    <gazebo reference="${namespace}/thruster_${thruster_id}">
+      <selfCollide>false</selfCollide>
+    </gazebo>
     <!-- Set up hydrodynamic plugin -->
     <gazebo>

Commit message: dynamics added

File: glider_hybrid_whoi_description/urdf/glider_hybrid_whoi_base_kinematics.xacro (robot description, xacro)
@@ -19,5 +19,9 @@
   <xacro:include filename="$(find uuv_gazebo_ros_plugins)/urdf/snippets.xacro"/>
   <!-- Properties -->
-  <xacro:property name="mass" value="10000.0"/>
+  <xacro:property name="mass" value="56.0"/>
+  <xacro:property name="fluid_density" value="1024.0"/>
+  <xacro:property name="gravity" value="9.81"/>
+  <xacro:property name="cob" value="0 0 0"/>
+  <xacro:property name="cog" value="0 0 0.0054"/>
   <xacro:property name="visual_mesh_file" value="file://$(find glider_hybrid_whoi_description)/mesh/glider_hybrid_whoi/glider_hybrid_whoi_body.dae" />
   <xacro:property name="collision_mesh_file" value="file://$(find glider_hybrid_whoi_description)/mesh/glider_hybrid_whoi/glider_hybrid_whoi_collision.dae" />
@@ -25,4 +29,5 @@
   <xacro:property name="right_prop_mesh_file" value="file://$(find glider_hybrid_whoi_description)/mesh/glider_hybrid_whoi/glider_hybrid_whoi_right_propeller.dae" />
   <xacro:macro name="glider_hybrid_whoi_base" params="namespace debug inertial_reference_frame">
+    <!-- Base_link of the model -->
     <link name="${namespace}/base_link">
       <visual>
@@ -41,8 +46,32 @@
         <mass value="${mass}"/>
         <origin xyz="0 0 0" rpy="0 0 0" />
-        <inertia ixx="30.0" ixy="0" ixz="0" iyy="0.6" iyz="0" izz="5.0" />
+        <inertia ixx="0.3048" ixy="0" ixz="0" iyy="13.976" iyz="0" izz="13.976" />
       </inertial>
     </link>
-  <xacro:property name="thruster_id" value="1"/>
+    <!-- Dummy propeller plugin properties (rotorConstant = 0) -->
+    <!-- This is for topics used to visualize the propeller roatation  -->
+    <xacro:property name="dummy_plugin_properties_for_visual_rotation">
+      <dynamics>
+        <type>FirstOrder</type>
+        <timeConstant>0.0</timeConstant>
+      </dynamics>
+      <conversion>
+        <type>Basic</type>
+        <rotorConstant>0.0</rotorConstant>
+      </conversion>
+    </xacro:property>
+    <xacro:property name="dummy_link_properties_for_visual_rotation">
+      <xacro:box_inertial x="0" y="0" z="0" mass="0.00001">
+        <origin xyz="0 0 0" rpy="0 0 0"/>
+      </xacro:box_inertial>
+      <collision>
+        <geometry>
+          <cylinder length="0.000001" radius="0.000001"/>
+        </geometry>
+        <origin xyz="0 0 0" rpy="0 0 0"/>
+      </collision>
+    </xacro:property>
+    <!-- First propeller -->
+    <xacro:property name="thruster_id" value="1"/>
     <joint name="${namespace}/thruster_${thruster_id}_joint" type="continuous">
       <origin xyz="-0.558 -0.05 0" rpy="0 0 -${0.07*pi}"/>
@@ -52,7 +81,5 @@
     </joint>
     <link name="${namespace}/thruster_${thruster_id}">
-      <xacro:box_inertial x="0" y="0" z="0" mass="0.00001">
-        <origin xyz="0 0 0" rpy="0 0 0"/>
-      </xacro:box_inertial>
+      <xacro:insert_block name="dummy_link_properties_for_visual_rotation"/>
       <visual>
         <origin xyz="0.541 0.12 0" rpy="0 0 -${0.46*pi}"/>
@@ -61,10 +88,4 @@
         </geometry>
       </visual>
-      <collision>
-        <geometry>
-          <cylinder length="0.000001" radius="0.000001"/>
-        </geometry>
-        <origin xyz="0 0 0" rpy="0 0 0"/>
-      </collision>
     </link>
     <gazebo>
@@ -73,12 +94,5 @@
         <jointName>${namespace}/thruster_${thruster_id}_joint</jointName>
         <thrusterID>${thruster_id}</thrusterID>
-        <dynamics>
-          <type>FirstOrder</type>
-          <timeConstant>0.0</timeConstant>
-        </dynamics>
-        <conversion>
-          <type>Basic</type>
-          <rotorConstant>0.0</rotorConstant>
-        </conversion>
+        <xacro:insert_block name="dummy_plugin_properties_for_visual_rotation"/>
       </plugin>
     </gazebo>
@@ -86,4 +100,5 @@
       <selfCollide>false</selfCollide>
     </gazebo>
+    <!-- Second propeller -->
     <xacro:property name="thruster_id" value="0"/>
     <joint name="${namespace}/thruster_${thruster_id}_joint" type="continuous">
@@ -94,7 +109,5 @@
     </joint>
     <link name="${namespace}/thruster_${thruster_id}">
-      <xacro:box_inertial x="0" y="0" z="0" mass="0.00001">
-        <origin xyz="0 0 0" rpy="0 0 0"/>
-      </xacro:box_inertial>
+      <xacro:insert_block name="dummy_link_properties_for_visual_rotation"/>
       <visual>
         <origin xyz="-0.541 0.12 0" rpy="0 0 ${0.46*pi}"/>
@@ -103,10 +116,4 @@
         </geometry>
       </visual>
-      <collision>
-        <geometry>
-          <cylinder length="0.000001" radius="0.000001"/>
-        </geometry>
-        <origin xyz="0 0 0" rpy="0 0 0"/>
-      </collision>
     </link>
     <gazebo>
@@ -115,12 +122,5 @@
         <jointName>${namespace}/thruster_${thruster_id}_joint</jointName>
         <thrusterID>${thruster_id}</thrusterID>
-        <dynamics>
-          <type>FirstOrder</type>
-          <timeConstant>0.0</timeConstant>
-        </dynamics>
-        <conversion>
-          <type>Basic</type>
-          <rotorConstant>0.0</rotorConstant>
-        </conversion>
+        <xacro:insert_block name="dummy_plugin_properties_for_visual_rotation"/>
       </plugin>
     </gazebo>
@@ -128,9 +128,37 @@
       <selfCollide>false</selfCollide>
     </gazebo>
-    <!-- Set up hydrodynamic plugin -->
+    <!-- Kinematics Plugin -->
     <gazebo>
       <plugin name="${namespace}_direct_kinematics_plugin"
               filename="libdirect_kinematics_ros_plugin.so">
-        <writeLog>1</writeLog>
+        <fluid_deisnty>${fluid_density}</fluid_deisnty>
+        <writeLog>true</writeLog>
+        <flow_velocity_topic>/hydrodynamics/current_velocity</flow_velocity_topic>
+        <use_global_ocean_current>true</use_global_ocean_current>
+        <!-- Dynamics properties -->
+        <apply_dynamics>true</apply_dynamics>
+        <dynamics>
+          <hull_mass>48.2</hull_mass>
+          <hull_length>2.0</hull_length>
+          <hull_radius>0.105</hull_radius>
+          <shifter_mass>7.8</shifter_mass>
+          <ballast_radius>0.07</ballast_radius>
+          <default_mass_position>0.4</default_mass_position>
+          <default_ballast_position>0.711</default_ballast_position>
+          <initial_mass_position>-0.018</initial_mass_position>
+          <initial_ballast_position>-0.01024</initial_ballast_position>
+          <max_mass_position>0.03</max_mass_position>
+          <max_ballast_volume>2.4e-04</max_ballast_volume>
+          <center_of_buoyancy>0 0 0</center_of_buoyancy>
+          <center_of_gravity>0 0 0.0054</center_of_gravity>
+          <linear_damping>
+            0       0       0       0       0       0
+            0       0       0       0       0       0
+            0       0       -14     0       0       0
+            0       0       0       0       0       0
+            0       0       0       0       -12     0
+            0       0       0       0       0       0
+          </linear_damping>
+        </dynamics>
       </plugin>
     </gazebo>

File: glider_hybrid_whoi_description/urdf/glider_hybrid_whoi_base_test.xacro (robot description, xacro)
@@ -42,5 +42,5 @@
     <link name="${namespace}/base_link">
       <visual>
-        <origin xyz="0 0 0" rpy="0 0 -1.5708" />
+        <origin xyz="0 0 0" rpy="0 0 -${0.5*pi}" />
         <geometry>
           <mesh filename="${visual_mesh_file}" scale="1 1 1" />
@@ -48,5 +48,5 @@
       </visual>
       <collision>
-        <origin xyz="0 0 0" rpy="0 0 -1.5708" />
+        <origin xyz="0 0 0" rpy="0 0 -${0.5*pi}" />
         <geometry>
           <mesh filename="${collision_mesh_file}" scale="1 1 1" />
@@ -59,43 +59,88 @@
       </inertial>
     </link>
-    <link name="${namespace}/left_propeller_link">
+    <xacro:property name="thruster_id" value="1"/>
+    <joint name="${namespace}/thruster_${thruster_id}_joint" type="continuous">
+      <origin xyz="-0.558 -0.05 0" rpy="0 0 -${0.07*pi}"/>
+      <axis xyz="1 0 0"/>
+      <parent link="${namespace}/base_link"/>
+      <child link="${namespace}/thruster_${thruster_id}"/>
+    </joint>
+    <link name="${namespace}/thruster_${thruster_id}">
+      <xacro:box_inertial x="0" y="0" z="0" mass="0.00001">
+        <origin xyz="0 0 0" rpy="0 0 0"/>
+      </xacro:box_inertial>
       <visual>
-        <origin xyz="0 0 0" rpy="0 0 0 " />
-        <geometry>
-          <mesh filename="${left_prop_mesh_file}" scale="1 1 1" />
+        <origin xyz="0.541 0.12 0" rpy="0 0 -${0.46*pi}"/>
+        <geometry>
+          <mesh filename="${right_prop_mesh_file}" scale="1 1 1"/>
         </geometry>
       </visual>
+      <collision>
+        <geometry>
+          <cylinder length="0.000001" radius="0.000001"/>
+        </geometry>
+        <origin xyz="0 0 0" rpy="0 0 0"/>
+      </collision>
     </link>
-    <joint name="${namespace}/left_propeller_joint" type="continuous">
-      <origin xyz="0 0 0" rpy="0 0 0" />
+    <gazebo>
+      <plugin name="${namespace}_${thruster_id}_thruster_model" filename="libuuv_thruster_ros_plugin.so">
+        <linkName>${namespace}/thruster_${thruster_id}</linkName>
+        <jointName>${namespace}/thruster_${thruster_id}_joint</jointName>
+        <thrusterID>${thruster_id}</thrusterID>
+        <dynamics>
+          <type>FirstOrder</type>
+          <timeConstant>0.0</timeConstant>
+        </dynamics>
+        <conversion>
+          <type>Basic</type>
+          <rotorConstant>0.0</rotorConstant>
+        </conversion>
+      </plugin>
+    </gazebo>
+    <gazebo reference="${namespace}/thruster_${thruster_id}">
+      <selfCollide>false</selfCollide>
+    </gazebo>
+    <xacro:property name="thruster_id" value="0"/>
+    <joint name="${namespace}/thruster_${thruster_id}_joint" type="continuous">
+      <origin xyz="-0.558 0.05 0" rpy="0 0 ${0.07*pi+pi}"/>
+      <axis xyz="1 0 0"/>
       <parent link="${namespace}/base_link"/>
-      <child link="${namespace}/left_propeller_link"/>
-      <axis xyz="0 1 0" />
+      <child link="${namespace}/thruster_${thruster_id}"/>
     </joint>
-    <link name="${namespace}/right_propeller_link">
+    <link name="${namespace}/thruster_${thruster_id}">
+      <xacro:box_inertial x="0" y="0" z="0" mass="0.00001">
+        <origin xyz="0 0 0" rpy="0 0 0"/>
+      </xacro:box_inertial>
       <visual>
-        <origin xyz="0 0 0" rpy="0 0 0" />
-        <geometry>
-          <mesh filename="${right_prop_mesh_file}" scale="1 1 1" />
+        <origin xyz="-0.541 0.12 0" rpy="0 0 ${0.46*pi}"/>
+        <geometry>
+          <mesh filename="${left_prop_mesh_file}" scale="1 1 1"/>
         </geometry>
       </visual>
+      <collision>
+        <geometry>
+          <cylinder length="0.000001" radius="0.000001"/>
+        </geometry>
+        <origin xyz="0 0 0" rpy="0 0 0"/>
+      </collision>
     </link>
-    <joint name="${namespace}/right_propeller_joint" type="continuous">
-      <origin xyz="0 0 0" rpy="0 0 0" />
-      <parent link="${namespace}/base_link"/>
-      <child link="${namespace}/right_propeller_link"/>
-      <axis xyz="0 1 0" />
-    </joint>
-    <link name='${namespace}/battery_link2'>
-      <origin xyz="0 0 0" rpy="0 0 0" />
-      <battery name='${namespace}/battery'>
-        <voltage>4.2</voltage>
-      </battery>
-    </link>
-    <joint name='${namespace}/battery_joint2' type='fixed'>
-      <origin xyz="0 0 0" rpy="0 0 0" />
-      <parent link="${namespace}/base_link"/>
-      <child link="${namespace}/battery_link2"/>
-    </joint>
+    <gazebo>
+      <plugin name="${namespace}_${thruster_id}_thruster_model" filename="libuuv_thruster_ros_plugin.so">
+        <linkName>${namespace}/thruster_${thruster_id}</linkName>
+        <jointName>${namespace}/thruster_${thruster_id}_joint</jointName>
+        <thrusterID>${thruster_id}</thrusterID>
+        <dynamics>
+          <type>FirstOrder</type>
+          <timeConstant>0.0</timeConstant>
+        </dynamics>
+        <conversion>
+          <type>Basic</type>
+          <rotorConstant>0.0</rotorConstant>
+        </conversion>
+      </plugin>
+    </gazebo>
+    <gazebo reference="${namespace}/thruster_${thruster_id}">
+      <selfCollide>false</selfCollide>
+    </gazebo>
     <!-- Set up hydrodynamic plugin -->
     <gazebo>
@@ -110,8 +155,8 @@
           <center_of_gravity>${cog}</center_of_gravity>
           <neutrally_buoyant>0</neutrally_buoyant>
-          <hard_code_input>1</hard_code_input>
+          <hard_code_input>0</hard_code_input>
           <hydrodynamic_model>
             <type>fossen</type>
-            <added_mass> <!-- dummy input. The values will be changed within glider kinamatics plugin-->
+            <added_mass> <!-- dummy input. The values will be changed within glider dynamics plugin-->
               100 0   0   0   0   0
               0   100 0   0   0   0

Commit message: thruster coefficient definable at sdf

File: glider_hybrid_whoi_description/urdf/glider_hybrid_whoi_base_kinematics.xacro (robot description, xacro)
@@ -141,29 +141,10 @@
         <C_D>0.2534</C_D>
         <C_L>0.4160</C_L>
-        <!-- Dynamics properties -->
-        <use_dynamics>false</use_dynamics>
-        <dynamics>
-          <hull_mass>48.2</hull_mass>
-          <hull_length>2.0</hull_length>
-          <hull_radius>0.105</hull_radius>
-          <shifter_mass>7.8</shifter_mass>
-          <ballast_radius>0.07</ballast_radius>
-          <default_mass_position>0.4</default_mass_position>
-          <default_ballast_position>0.711</default_ballast_position>
-          <initial_mass_position>-0.018</initial_mass_position>
-          <initial_ballast_position>-0.01024</initial_ballast_position>
-          <max_mass_position>0.03</max_mass_position>
-          <max_ballast_volume>2.4e-04</max_ballast_volume>
-          <center_of_buoyancy>0 0 0</center_of_buoyancy>
-          <center_of_gravity>0 0 0.0054</center_of_gravity>
-          <linear_damping>
-            0       0       0       0       0       0
-            0       0       0       0       0       0
-            0       0       -14     0       0       0
-            0       0       0       0       0       0
-            0       0       0       0       -12     0
-            0       0       0       0       0       0
-          </linear_damping>
-        </dynamics>
+        <f_thruster_voltage_v1>1.8953</f_thruster_voltage_v1>
+        <f_thruster_voltage_v2>-1.995</f_thruster_voltage_v2>
+        <f_thruster_voltage_v3>1.8701</f_thruster_voltage_v3>
+        <f_thruster_power_w1>-0.020919</f_thruster_power_w1>
+        <f_thruster_power_w2>1.4699</f_thruster_power_w2>
+        <f_thruster_power_w3>0.97895</f_thruster_power_w3>
       </plugin>
     </gazebo>

Commit message: Pitch based on dynamics calculation

File: glider_hybrid_whoi_description/urdf/glider_hybrid_whoi_base_kinematics.xacro (robot description, xacro)
@@ -148,4 +148,30 @@
         <f_thruster_power_w2>1.4699</f_thruster_power_w2>
         <f_thruster_power_w3>0.97895</f_thruster_power_w3>
+        <!-- Dynamics properties -->
+        <use_dynamics>true</use_dynamics>
+        <hard_code_input>true</hard_code_input>
+        <dynamics>
+          <hull_mass>48.2</hull_mass>
+          <hull_length>2.0</hull_length>
+          <hull_radius>0.105</hull_radius>
+          <shifter_mass>7.8</shifter_mass>
+          <ballast_radius>0.07</ballast_radius>
+          <default_mass_position>0.4</default_mass_position>
+          <default_ballast_position>0.711</default_ballast_position>
+          <initial_mass_position>-0.018</initial_mass_position>
+          <initial_ballast_position>-0.01024</initial_ballast_position>
+          <max_mass_position>0.03</max_mass_position>
+          <max_ballast_volume>2.4e-04</max_ballast_volume>
+          <center_of_buoyancy>0 0 0</center_of_buoyancy>
+          <center_of_gravity>0 0 0.0054</center_of_gravity>
+          <linear_damping>
+            0       0       0       0       0       0
+            0       0       0       0       0       0
+            0       0       -14     0       0       0
+            0       0       0       0       0       0
+            0       0       0       0       -12     0
+            0       0       0       0       0       0
+          </linear_damping>
+        </dynamics>
       </plugin>
       <plugin name="{namespace}_dave_ocean_current_plugin" filename="libdave_ocean_current_model_plugin.so">
@@ -167,5 +193,5 @@
           </velocity_down>
         </transient_current>
-        <tide_oscillation>true</tide_oscillation>
+        <tide_oscillation>false</tide_oscillation>
       </plugin>
     </gazebo>
